File: Schematic/PowerInput/PowerInput.kicad_pcb (KiCad board)
At the start: 2 copper layers, 70 x 40 mm, 26 parts, among them J101 PSU1 Pri, J102 PSU2 Pri, J103 PSU1 Sec, J104 PSU2 Sec, J105 Power LED, J106 230VAC In, J107 Power switch, J108 To MainBoard, J109 To Heater PSU

Commit message: Minor layout changes
Parts:
- turned D102 to -90 degrees
Routing:
- net Net-(D102-Pad2): track 2.92 -> 6.07 mm
- net /PSU2_0V: track 21.1 -> 22.2 mm
Changed lines of the file:
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@@
   )
   (footprint "LED_SMD:LED_0805_2012Metric_Pad1.15x1.40mm_HandSolder" (layer "F.Cu")
-    (at 136.5 74 90)
+    (at 136.5 74 -90)
     (descr "LED SMD 0805 (2012 Metric), square (rectangular) end terminal, IPC_7351 nominal, (Body size source: https://docs.google.com/spreadsheets/d/1BsfQQcO9C6DZCsRaXUlFlo91Tg2WpOkGARC1WS5S8t0/edit?usp=sharing), generated with kicad-footprint-generator")
     (tags "LED handsolder")
@@
     (property "Sheetname" "")
     (attr smd)
-    (fp_text reference "D102" (at 0 -1.85 90) (layer "F.SilkS")
+    (fp_text reference "D102" (at 0 1.75 90) (layer "F.SilkS")
       (effects (font (size 1 1) (thickness 0.15)))
     )
@@
     (fp_line (start 1 0.6) (end 1 -0.6) (layer "F.Fab") (width 0.1))
     (fp_line (start -1 0.6) (end 1 0.6) (layer "F.Fab") (width 0.1))
-    (pad "1" smd roundrect (at -1.025 0 90) (size 1.15 1.4) (layers "F.Cu" "F.Paste" "F.Mask") (roundrect_rratio 0.2173913043)
+    (pad "1" smd roundrect (at -1.025 0 270) (size 1.15 1.4) (layers "F.Cu" "F.Paste" "F.Mask") (roundrect_rratio 0.2173913043)
       (net 5 "/PSU2_0V") (pinfunction "K") (pintype "passive"))
-    (pad "2" smd roundrect (at 1.025 0 90) (size 1.15 1.4) (layers "F.Cu" "F.Paste" "F.Mask") (roundrect_rratio 0.2173913043)
+    (pad "2" smd roundrect (at 1.025 0 270) (size 1.15 1.4) (layers "F.Cu" "F.Paste" "F.Mask") (roundrect_rratio 0.2173913043)
       (net 6 "Net-(D102-Pad2)") (pinfunction "A") (pintype "passive"))
     (model "${KICAD6_3DMODEL_DIR}/LED_SMD.3dshapes/LED_0805_2012Metric.wrl"
@@
   (segment (start 136.5 60.45) (end 136.5 57.025) (width 0.25) (layer "F.Cu") (net 4))
   (segment (start 130.5 78) (end 127 81.5) (width 1) (layer "F.Cu") (net 5))
-  (segment (start 133.525 78) (end 130.5 78) (width 0.25) (layer "F.Cu") (net 5))
   (segment (start 123 81.46) (end 119.54 78) (width 1) (layer "F.Cu") (net 5))
+  (segment (start 135.315 72.975) (end 130.29 78) (width 0.25) (layer "F.Cu") (net 5))
   (segment (start 127 81.5) (end 123 81.5) (width 1) (layer "F.Cu") (net 5))
   (segment (start 123 81.5) (end 123 81.46) (width 1) (layer "F.Cu") (net 5))
-  (segment (start 136.5 75.025) (end 133.525 78) (width 0.25) (layer "F.Cu") (net 5))
-  (segment (start 136.5 72.975) (end 136.5 70.05) (width 0.25) (layer "F.Cu") (net 6))
+  (segment (start 136.5 72.975) (end 135.315 72.975) (width 0.25) (layer "F.Cu") (net 5))
+  (segment (start 136.5 75.025) (end 136.5 74.987437) (width 0.25) (layer "F.Cu") (net 6))
+  (segment (start 137.825 73.662437) (end 137.825 71.375) (width 0.25) (layer "F.Cu") (net 6))
+  (segment (start 136.5 74.987437) (end 137.825 73.662437) (width 0.25) (layer "F.Cu") (net 6))
+  (segment (start 137.825 71.375) (end 136.5 70.05) (width 0.25) (layer "F.Cu") (net 6))
   (segment (start 81.96 51) (end 81.96 57.4015) (width 1) (layer "B.Cu") (net 7))
   (segment (start 81.96 57.4015) (end 84.5 59.9415) (width 1) (layer "B.Cu") (net 7))

Commit message: Added filtering on PSU1 secondary
Parts:
- added C102: 220µF 35V, Capacitor_THT:CP_Radial_D10.0mm_P7.50mm, F.Cu at (153.1, 65.0)
- added FB101: FerriteBead, Inductor_SMD:L_1812_4532Metric_Pad1.30x3.40mm_HandSolder, F.Cu at (144.2, 80.6)
- added FB102: FerriteBead, Inductor_SMD:L_1812_4532Metric_Pad1.30x3.40mm_HandSolder, F.Cu at (128.4, 80.6)
- added L101: 330µH 3.3A, Inductor_THT:L_Radial_D24.4mm_P23.70mm_Murata_1400series, F.Cu at (148.3, 65.0)
- F102: renamed from F101; value T1A -> T3.15A
- G***: moved to F.Cu
- R102: value 1kΩ 1/2W -> 3.9kΩ 1/2W
- moved J106 61.6 mm to (166.2, 68.3), turned to 180 degrees
- moved R102 56.5 mm to (165.4, 61.4), turned to 0 degrees
- moved H103 30.1 mm to (166.6, 48.5)
- moved H104 30.1 mm to (166.6, 81.5)
- moved R103 29.2 mm to (165.4, 73.0), turned to 0 degrees
- moved R101 29.2 mm to (165.4, 57.4), turned to 0 degrees
- moved J109 29.0 mm to (154.2, 78.2)
- moved J104 29.0 mm to (159.3, 52.0)
- moved D102 28.6 mm to (165.0, 76.8), turned to 0 degrees
- moved D101 28.6 mm to (165.0, 53.4), turned to 0 degrees
- moved G*** 19.5 mm to (136.6, 48.8), turned to 0 degrees
- moved F103 12.0 mm to (107.6, 65.0)
- moved F101 11.0 mm to (119.5, 65.0)
- renumbered F102 to F101, J108 to J104, J106 to J105, J105 to J106, J104 to J108
Connections:
- D102 pad 1: /PSU2_0V -> /HeaterPSU_0V
- F101 pad 1: /PSU1_19V -> Net-(F101-Pad1)
- F101 pad 2: Net-(F102-Pad2) -> /PSU1_19V
- F103 pad 1: /PSU2_19V -> Net-(F103-Pad1)
- F103 pad 2: Net-(F103-Pad2) -> /PSU2_19V
- J103 pad 1: Net-(F102-Pad2) -> Earth
- J103 pad 2: Earth -> /PSU1_19V
- J104 pad 1: /PSU1_19V -> Earth
- J104 pad 2: Earth -> /MainBoard_19V
- J108 pad 1: Net-(F103-Pad2) -> /PSU2_19V
- J109 pad 1: /PSU2_19V -> /HeaterPSU_19V
- J109 pad 2: /PSU2_0V -> /HeaterPSU_0V
- R101 pad 1: /PSU1_19V -> /MainBoard_19V
- R102 pad 1: /PSU1_19V -> /MainBoard_19V
- R103 pad 1: /PSU2_19V -> /HeaterPSU_19V
Routing:
- net Earth: track 94.7 -> 141.4 mm
- net Net-(F103-Pad1): track 0.00 -> 41.0 mm
- net /HeaterPSU_0V: track 0.00 -> 37.2 mm
- net /MainBoard_19V: track 0.00 -> 34.4 mm, vias 0 -> 1
- net /PSU1_19V: track 43.2 -> 13.0 mm
- net /HeaterPSU_19V: track 0.00 -> 20.6 mm
- net Net-(F102-Pad2): track 14.9 -> 0.00 mm
- net /PSU2_0V: track 22.2 -> 7.71 mm
- net /PSU2_19V: track 31.2 -> 18.0 mm
- net Net-(F103-Pad2): track 12.5 -> 0.00 mm
- net Net-(F101-Pad1): track 0.00 -> 5.11 mm
- net Net-(D102-Pad2): track 6.07 -> 4.18 mm
- net Net-(D101-Pad2): track 3.43 -> 4.38 mm
Other:
- board size 70 x 40 mm -> 100 x 40 mm
- board text added: "+MB_PSU-"
- board text added: "+PSU1 Sec-"
- board text added: "- +"
- board text added: "µTracer Power Input 22_43_0121B Bjørner Sandom"
- board text removed: "+"
- board text removed: "-"
- board text removed: "-MB_PSU+"
- board text removed: "-PSU1 Sec+"
- board text removed: "PSU1"
- board text removed: "PSU2"
- board text removed: "µTracer Power Input 22_43_0121 Bjørner Sandom"
