File: Schematic/HeaterPSU_Digital/HeaterPSU_Digital.kicad_pcb (KiCad board)
At the start: 2 copper layers, 100 x 35 mm, 76 parts, among them J1 SMPS2_SEC, J2 Heater output, J3 Conn_01x06, Q1 IRF4905, Q2 SIRA24DP, U1 XL4005, U2 ADA4522-2, U3 MCP4726, U4 TPS54302, U5 INA293B1QDBVRQ1, U6 MCP4726, U7 INA219AIDCNR

Commit message: Added driver stage for output MOSFET
Parts:
- added D7: 12V, Diode_SMD:D_SOD-123, B.Cu at (148.1, 54.5)
- added Q3: BC847, Package_TO_SOT_SMD:SOT-23, B.Cu at (139.5, 60.5)
- added Q4: BC847, Package_TO_SOT_SMD:SOT-23, B.Cu at (134.7, 60.5)
- added R9: 1.5kΩ, Resistor_SMD:R_0603_1608Metric_Pad0.98x0.95mm_HandSolder, B.Cu at (134.7, 57.0)
- moved R14 19.5 mm to (138.1, 68.0), turned to 90 degrees
- moved D6 15.6 mm to (140.7, 68.0), turned to 90 degrees
- moved R10 5.12 mm to (139.3, 57.0), turned to 0 degrees
- renumbered D7 to D8, D8 to D9, R13 to R10, R9 to R11, R10 to R12, R11 to R13, R12 to R14, R14 to R15, R15 to R16, R16 to R17, R17 to R18, R18 to R19, R19 to R20, R20 to R21
Connections:
- Q2 pad 2: OUT_EN -> Net-(R10-Pad2)
- R10 pad 1: OUT_EN -> VDC
- R10 pad 2: GNDPWR -> Net-(R10-Pad2)
Routing:
- net VDC: track 91.1 -> 131.0 mm
- net Net-(R10-Pad2): track 0.00 -> 11.0 mm
- net OUT_EN: track 30.5 -> 21.7 mm
- net +5V: track 98.7 -> 106.8 mm, vias 5 -> 6
- net Net-(Q3-Pad1): track 0.00 -> 6.80 mm
- net Net-(C1-Pad1): track 37.3 -> 38.9 mm
- net GNDPWR: track 36.1 -> 34.9 mm, vias 86 -> 85
