File: Schematic/HeaterPSU/HeaterPSU.kicad_sch (KiCad schematic)
At the start: 65 parts, among them J201 Heater output, J202 To MCU Board, J203 SMPS2_SEC, Q201 SIRA24DP, Q202 IRF4905, SW201 ALPSALPINE_SRBV_1P5T, U201 XL4005, U202 MCP14A0052T, U203 INA293B, U204 L78L05_SOT89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

Commit message: Added project pictures
Parts:
- R216: value 82kΩ -> 91kΩ
Changed lines of the file:
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@@
     (in_bom yes) (on_board yes)
     (property "Reference" "R216" (id 0) (at 137.16 120.65 90))
-    (property "Value" "82kΩ" (id 1) (at 137.16 122.555 90))
+    (property "Value" "91kΩ" (id 1) (at 137.16 122.555 90))
     (property "Footprint" "Resistor_SMD:R_0603_1608Metric_Pad0.98x0.95mm_HandSolder" (id 2) (at 137.16 126.238 90)
       (effects (font (size 1.27 1.27)) hide)
@@
     )
     (path "/8388cf02-b7a0-4c05-bcd2-d3a51205ca58"
-      (reference "R216") (unit 1) (value "82kΩ") (footprint "Resistor_SMD:R_0603_1608Metric_Pad0.98x0.95mm_HandSolder")
+      (reference "R216") (unit 1) (value "91kΩ") (footprint "Resistor_SMD:R_0603_1608Metric_Pad0.98x0.95mm_HandSolder")
     )
     (path "/abaa147c-f464-4236-8a4d-0ce77003cf6c"

Commit message: Changed component values
Parts:
- R218, R220: value 3.9kΩ 1/2W -> 5.6kΩ 1/2W
Changed lines of the file:
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@@
       (effects (font (size 1.27 1.27)) (justify right))
     )
-    (property "Value" "3.9kΩ 1/2W" (id 1) (at 66.2686 177.673 0)
+    (property "Value" "5.6kΩ 1/2W" (id 1) (at 66.2686 177.673 0)
       (effects (font (size 1.27 1.27)) (justify right))
     )
@@
       (effects (font (size 1.27 1.27)) (justify right))
     )
-    (property "Value" "3.9kΩ 1/2W" (id 1) (at 31.3436 168.148 0)
+    (property "Value" "5.6kΩ 1/2W" (id 1) (at 31.3436 168.148 0)
       (effects (font (size 1.27 1.27)) (justify right))
     )
@@
     )
     (path "/f967a966-4ece-4602-ba4b-63d93cb59cbf"
-      (reference "R218") (unit 1) (value "3.9kΩ 1/2W") (footprint "Resistor_SMD:R_1210_3225Metric_Pad1.30x2.65mm_HandSolder")
+      (reference "R218") (unit 1) (value "5.6kΩ 1/2W") (footprint "Resistor_SMD:R_1210_3225Metric_Pad1.30x2.65mm_HandSolder")
     )
     (path "/a41f1dc4-7ce8-4d54-a1e4-c64a4d09b61d"
@@
     )
     (path "/d8009b04-9e5a-4dee-a875-459ac83c9f82"
-      (reference "R220") (unit 1) (value "3.9kΩ 1/2W") (footprint "Resistor_SMD:R_1210_3225Metric_Pad1.30x2.65mm_HandSolder")
+      (reference "R220") (unit 1) (value "5.6kΩ 1/2W") (footprint "Resistor_SMD:R_1210_3225Metric_Pad1.30x2.65mm_HandSolder")
     )
     (path "/5475ee01-b699-4c77-9e3c-aebe58d2969e"

Commit message: Added BOM (bill of materials)
Parts:
- SW201: value ALPSALPINE_SRBV_1P5T -> ALPSALPINE SRBV150901
Changed lines of the file:
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@@
     (in_bom yes) (on_board yes)
     (property "Reference" "SW201" (id 0) (at 97.155 70.485 0))
-    (property "Value" "ALPSALPINE_SRBV_1P5T" (id 1) (at 99.06 73.025 0))
+    (property "Value" "ALPSALPINE SRBV150901" (id 1) (at 99.06 73.025 0))
     (property "Footprint" "myDevices:SRBV141404" (id 2) (at 95.25 69.85 0)
       (effects (font (size 1.27 1.27)) hide)
@@
     )
     (path "/ae48d68f-db89-4dfb-be12-01fc736dda99"
-      (reference "SW201") (unit 1) (value "ALPSALPINE_SRBV_1P5T") (footprint "myDevices:SRBV141404")
+      (reference "SW201") (unit 1) (value "ALPSALPINE SRBV150901") (footprint "myDevices:SRBV141404")
     )
     (path "/a68274cb-50bb-431a-a8ea-e6aff6f46e70"
